Commit message: 10th week changes

File: turtlebot_sim/turtlebot2/urdf/turtlebot2.urdf (robot description, URDF)
Before this commit: robot turtlebot2, 24 links, 23 joints
Links:
- link base_link: geometry collision cylinder length=0.10938 radius=0.178; visual mesh filename=/home/tapi1300/ros2_humble/src/ThirdParty/kobuki_ros/kobuki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
- link wheel_left_link: geometry collision cylinder length=0.0206 radius=0.035; visual mesh filename=/home/tapi1300/ros2_humble/src/ThirdParty/kobuki_ros/kobuki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
- link wheel_right_link: geometry collision cylinder length=0.0206 radius=0.035; visual mesh filename=/home/tapi1300/ros2_humble/src/ThirdParty/kobuki_ros/kobuki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

Commit message: 12th week updates

File: turtlebot_sim/turtlebot2/urdf/turtlebot2.urdf (robot description, URDF)
Before this commit: robot turtlebot2, 24 links, 23 joints
Links:
- link base_link: geometry collision cylinder length=0.10938 radius=0.178; visual mesh filename=model://kobuki_description/share/kobuki_description/meshes/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
- link wheel_left_link: geometry collision cylinder length=0.0206 radius=0.035; visual mesh filename=model://kobuki_description/share/kobuki_description/meshes/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
- link wheel_right_link: geometry collision cylinder length=0.0206 radius=0.035; visual mesh filename=model://kobuki_description/share/kobuki_description/meshes/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
